File: station/eagle/Regn Weather Station.sch (EAGLE design)
At the start: 6 parts

Commit message: Refactored PCB size and logos
Parts:
- ESP8226: value ESP8266HUZZAH -> (none)
Changed lines of the file:
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@@
 <part name="FRAME1" library="frames" library_urn="urn:adsk.eagle:library:229" deviceset="FRAME_A_L" device=""/>
 <part name="BMP180" library="regn" deviceset="BMP180" device="" package3d_urn="urn:adsk.eagle:package:22469/2"/>
-<part name="ESP8226" library="regn" deviceset="ESP8266HUZZAH" device="" value="ESP8266HUZZAH"/>
+<part name="ESP8226" library="regn" deviceset="ESP8266HUZZAH" device=""/>
 <part name="TSL2561" library="regn" deviceset="TSL2561" device="" package3d_urn="urn:adsk.eagle:package:22477/2"/>
 <part name="DHT22" library="RHT03_DHT-22_AM2302" deviceset="RHT03_DHT-22_AM2302" device="WIRED"/>

Commit message: PCB optimizations and refining
Parts:
- R1: device SparkFun-Resistors:10KOHM-0603-1/10W-1% -> SparkFun-Resistors:10KOHM-HORIZ-1/4W-1%
- renumbered ESP8226 to ESP8266
Changed lines of the file:
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@@
 <?xml version="1.0" encoding="utf-8"?>
 <!DOCTYPE eagle SYSTEM "eagle.dtd">
-<eagle version="9.0.0">
+<eagle version="9.0.1">
 <drawing>
 <settings>
@@
 <part name="FRAME1" library="frames" library_urn="urn:adsk.eagle:library:229" deviceset="FRAME_A_L" device=""/>
 <part name="BMP180" library="regn" deviceset="BMP180" device="" package3d_urn="urn:adsk.eagle:package:22469/2"/>
-<part name="ESP8226" library="regn" deviceset="ESP8266HUZZAH" device=""/>
+<part name="ESP8266" library="regn" deviceset="ESP8266HUZZAH" device=""/>
 <part name="TSL2561" library="regn" deviceset="TSL2561" device="" package3d_urn="urn:adsk.eagle:package:22477/2"/>
 <part name="DHT22" library="RHT03_DHT-22_AM2302" deviceset="RHT03_DHT-22_AM2302" device="WIRED"/>
 <part name="GND1" library="SparkFun-PowerSymbols" deviceset="GND" device=""/>
 <part name="GND3" library="SparkFun-PowerSymbols" deviceset="GND" device=""/>
-<part name="R1" library="SparkFun-Resistors" deviceset="10KOHM" device="-0603-1/10W-1%" value="10k"/>
+<part name="R1" library="SparkFun-Resistors" deviceset="10KOHM" device="-HORIZ-1/4W-1%" value="10k"/>
 <part name="SUPPLY1" library="SparkFun-PowerSymbols" deviceset="3.3V" device=""/>
 <part name="SUPPLY2" library="SparkFun-PowerSymbols" deviceset="3.3V" device=""/>
@@
 <instance part="FRAME1" gate="G$2" x="38.1" y="-96.52"/>
 <instance part="BMP180" gate="G$1" x="48.26" y="-30.48" rot="R180"/>
-<instance part="ESP8226" gate="G$1" x="0" y="0"/>
+<instance part="ESP8266" gate="G$1" x="0" y="0"/>
 <instance part="TSL2561" gate="G$1" x="53.34" y="35.56"/>
 <instance part="DHT22" gate="G$1" x="-50.8" y="12.7" rot="R180"/>
@@
 </segment>
 <segment>
-<pinref part="ESP8226" gate="G$1" pin="GND"/>
+<pinref part="ESP8266" gate="G$1" pin="GND"/>
 <pinref part="GND2" gate="1" pin="GND"/>
 <wire x1="20.32" y1="-22.86" x2="25.4" y2="-22.86" width="0.1524" layer="91"/>
@@
 <wire x1="-30.48" y1="10.16" x2="-35.56" y2="10.16" width="0.1524" layer="91"/>
 <wire x1="-35.56" y1="10.16" x2="-35.56" y2="2.54" width="0.1524" layer="91"/>
-<pinref part="ESP8226" gate="G$1" pin="#14"/>
+<pinref part="ESP8266" gate="G$1" pin="#14"/>
 <wire x1="-35.56" y1="2.54" x2="-20.32" y2="2.54" width="0.1524" layer="91"/>
 <pinref part="R1" gate="G$1" pin="1"/>
@@
 <pinref part="DHT22" gate="G$1" pin="VDD"/>
 <wire x1="-40.64" y1="5.08" x2="-40.64" y2="-2.54" width="0.1524" layer="91"/>
-<pinref part="ESP8226" gate="G$1" pin="#12"/>
+<pinref part="ESP8266" gate="G$1" pin="#12"/>
 <wire x1="-40.64" y1="-2.54" x2="-20.32" y2="-2.54" width="0.1524" layer="91"/>
 </segment>
@@
 </segment>
 <segment>
-<pinref part="ESP8226" gate="G$1" pin="3V"/>
+<pinref part="ESP8266" gate="G$1" pin="3V"/>
 <pinref part="SUPPLY4" gate="G$1" pin="3.3V"/>
 <wire x1="20.32" y1="-12.7" x2="25.4" y2="-12.7" width="0.1524" layer="91"/>
@@
 <wire x1="53.34" y1="-7.62" x2="35.56" y2="-7.62" width="0.1524" layer="91"/>
 <wire x1="35.56" y1="-7.62" x2="35.56" y2="7.62" width="0.1524" layer="91"/>
-<pinref part="ESP8226" gate="G$1" pin="#4"/>
+<pinref part="ESP8266" gate="G$1" pin="#4"/>
 <wire x1="35.56" y1="7.62" x2="20.32" y2="7.62" width="0.1524" layer="91"/>
 <pinref part="TSL2561" gate="G$1" pin="SDA"/>
@@
 <wire x1="48.26" y1="-2.54" x2="40.64" y2="-2.54" width="0.1524" layer="91"/>
 <wire x1="40.64" y1="-2.54" x2="40.64" y2="12.7" width="0.1524" layer="91"/>
-<pinref part="ESP8226" gate="G$1" pin="#5"/>
+<pinref part="ESP8266" gate="G$1" pin="#5"/>
 <wire x1="40.64" y1="12.7" x2="20.32" y2="12.7" width="0.1524" layer="91"/>
 <pinref part="TSL2561" gate="G$1" pin="SCL"/>
@@
 <net name="N$4" class="0">
 <segment>
-<pinref part="ESP8226" gate="G$1" pin="#16"/>
+<pinref part="ESP8266" gate="G$1" pin="#16"/>
 <wire x1="-20.32" y1="7.62" x2="-22.86" y2="7.62" width="0.1524" layer="91"/>
 <wire x1="-22.86" y1="7.62" x2="-22.86" y2="22.86" width="0.1524" layer="91"/>
-<pinref part="ESP8226" gate="G$1" pin="RST"/>
+<pinref part="ESP8266" gate="G$1" pin="RST"/>
 <wire x1="-22.86" y1="22.86" x2="-20.32" y2="22.86" width="0.1524" layer="91"/>
 </segment>
@@
 <segment>
 <pinref part="BATT" gate="G$1" pin="2"/>
-<pinref part="ESP8226" gate="G$1" pin="VBAT"/>
+<pinref part="ESP8266" gate="G$1" pin="VBAT"/>
 <wire x1="-33.02" y1="-17.78" x2="-20.32" y2="-17.78" width="0.1524" layer="91"/>
 </segment>
@@
 <wire x1="-33.02" y1="-20.32" x2="-25.4" y2="-20.32" width="0.1524" layer="91"/>
 <wire x1="-25.4" y1="-20.32" x2="-25.4" y2="-22.86" width="0.1524" layer="91"/>
-<pinref part="ESP8226" gate="G$1" pin="GND2"/>
+<pinref part="ESP8266" gate="G$1" pin="GND2"/>
 <wire x1="-25.4" y1="-22.86" x2="-20.32" y2="-22.86" width="0.1524" layer="91"/>
 </segment>
